Commit message: my robaka

File: urdf/robaka_v2_copy.xacro (robot description, xacro)
@@ -1,16 +1,13 @@
 <?xml version="1.0"?>
 <robot xmlns:xacro="http://www.ros.org/wiki/xacro" name="robaka_v2">
-  <xacro:property name="base_width" value="0.393"/>
-  <xacro:property name="base_len" value="0.490"/>
-  <xacro:property name="base_height" value="0.018"/>
-  <xacro:property name="base_width_1" value="0.393"/>
-  <xacro:property name="base_len_1" value="0.390"/>
-  <xacro:property name="base_height_1" value="0.150"/>
+  <xacro:property name="base_width" value="0.3"/>
+  <xacro:property name="base_len" value="0.4"/>
+  <xacro:property name="base_height" value="0.12"/>
   <xacro:property name="wheel_radius" value="0.085"/>
-  <xacro:property name="base_wheel_gap" value="0.01"/>
-  <xacro:property name="wheel_separation" value="0.307"/>
-  <xacro:property name="wheel_joint_offset" value="-0.150"/>
-  <xacro:property name="caster_wheel_radius" value="0.0475"/>
-  <xacro:property name="caster_wheel_joint_offset" value="0.1300"/>
+  <xacro:property name="base_wheel_gap" value="0.02"/>
+  <xacro:property name="wheel_separation" value="0.31"/>
+  <xacro:property name="wheel_joint_offset" value="-0.107"/>
+  <xacro:property name="caster_wheel_radius" value="0.0375"/>
+  <xacro:property name="caster_wheel_joint_offset" value="0.12"/>
   <xacro:include filename="$(find robaka)/urdf/robaka_v2_gazebo_plugins.xacro"/>
   <material name="blue">
@@ -40,7 +37,5 @@
     </inertial>
   </xacro:macro>
-<!--
   <link name="dummy"/>
--->
   <link name="base_footprint">
     <xacro:box_inertia m="8" w="0.001" h="0.001" d="0.001"/>
@@ -53,10 +48,8 @@
     </visual>
   </link>
-<!--
   <joint name="dummy_joint" type="fixed">
      <parent link="dummy"/>
      <child link="base_footprint"/>
-  </joint>
- -->
+     </joint>
   <link name="base_link">
     <xacro:box_inertia m="1" w="${base_len}" h="${base_width}" d="0.01"/>
@@ -78,23 +71,4 @@
     <child link="base_link" />
   </joint>
-  <link name="base_link_1">
-    <xacro:box_inertia m="1" w="${base_len_1}" h="${base_width_1}" d="0.01"/>
-    <visual>
-      <material name="lightgray"/>
-      <geometry>
-        <box size="${base_len_1} ${base_width_1} ${base_height_1}"/>
-      </geometry>
-    </visual>
-    <collision>
-      <geometry>
-        <box size="${base_len_1} ${base_width_1} ${base_height_1}"/>
-      </geometry>
-    </collision>
-  </link>
-  <joint name="base_link_joint_1" type="fixed">
-    <origin xyz="${-(base_len-base_len_1)/2} 0 ${wheel_radius}" rpy="0 0 0" />
-    <parent link="base_link"/>
-    <child link="base_link_1" />
-  </joint>
   <xacro:macro name="cylinder_inertia" params="m r h">
     <inertial>
@@ -113,5 +87,5 @@
       </visual>
       <collision>
-        <origin xyz="0 0 0" rpy="${pi/2} 0 0"/>0
+        <origin xyz="0 0 0" rpy="${pi/2} 0 0"/>
         <geometry>
           <cylinder radius="${wheel_radius}" length="0.02"/>
@@ -120,9 +94,9 @@
       <xacro:cylinder_inertia m="10" r="${wheel_radius}" h="0.02"/>
     </link>
-    <joint name="${prefix}_wheel_joint" type="continuous">
+    <joint name="${prefix}_wheel" type="continuous">
       <axis xyz="0 1 0" rpy="0 0 0" />
       <parent link="base_link"/>
       <child link="${prefix}_wheel"/>
-      <origin xyz="${wheel_joint_offset} ${((base_width/2)+base_wheel_gap)*reflect} 0" rpy="0 0 0"/>
+      <origin xyz="${wheel_joint_offset} ${((base_width/2)+base_wheel_gap)*reflect} -0.06" rpy="0 0 0"/>
     </joint>
   </xacro:macro>
@@ -155,7 +129,6 @@
     <parent link="base_link"/>
     <child link="caster_wheel"/>
-    <origin xyz="${caster_wheel_joint_offset} 0 -${caster_wheel_radius-0.006}" rpy="0 0 0"/>
+    <origin xyz="${caster_wheel_joint_offset} 0 -${0.06+caster_wheel_radius}" rpy="0 0 0"/>
   </joint>
-<!--
   <joint name="imu_joint" type="fixed">
     <parent link="base_link" />
@@ -164,9 +137,8 @@
   </joint>
   <link name="imu" />
-  -->
   <joint name="lidar_joint" type="fixed">
     <parent link="base_link" />
     <child link="lidar" />
-    <origin xyz="0.0 0.0 ${0.018+0.153+0.004}" rpy="0 0 3.14159" />
+    <origin xyz="0.0 0.0 0.12" rpy="0 0 3.14159" />
   </joint>
   <link name="lidar">
@@ -180,5 +152,5 @@
   </link>
   <joint name="camera_joint" type="fixed">
-    <origin xyz="0.185 0 ${0.025}" rpy="0 0 3.14159" />
+    <origin xyz="0.185 0 0.07" rpy="0 0 3.14159" />
     <parent link="base_link" />
     <child link="camera_link" />
